File: PCBs/Light Sensor/SensorBoard.brd (EAGLE design)
At the start: 70.6 x 56.8 mm, 36 parts, among them J1 AVR_SPI_PRG_6PTH, U2 MIC5219 3.3V

Commit message: Rev. B layout complete, design review soon
Parts:
- removed STANDOFF1, STANDOFF2, STANDOFF3: STAND-OFF, SparkFun-Electromechanical:STAND-OFF
- removed U$7: ATTINY84, SparkFun-DigitalIC:SO14
- removed U$8: SN74LVC2T45, MyLibrary:DCT-R-PDSO-G8
- added R6: 1k, rcl:R1210
- added U1: APDS-9008, MyLibrary:APDS-9008
- added U3: OPT101TH, MyLibrary:DIL08
- added U4: ATTINY84HANDSOLDER, MyLibrary:SO14-EZ
- C1: value 0.1uf -> 470pF
- C2: value 8.2pf -> 0.1uf
- C3: value 1.0uf -> 0.1uf
- C4: value 10uf -> 8.2pf
- C5: value 0.1uf -> 1.0uf
- C6: value 470pF -> 10uf
- R1: value 10 -> 1k; device SparkFun-Passives:AXIAL-0.3 -> rcl:R1210
- R2: value 1k -> 10; device rcl:R1210 -> SparkFun-Passives:AXIAL-0.3
- U$2: value APDS-9008 -> PROTOAREA-10X10; device MyLibrary:APDS-9008 -> MyLibrary:PROTOAREA-10X10
- U$3: value PROTOAREA-10X10 -> SN74LVC1T45; device MyLibrary:PROTOAREA-10X10 -> MyLibrary:DBV-R-PDSO-G6
- U$4: value OPT101TH -> SN74LVC1T45; device MyLibrary:DIL08 -> MyLibrary:DBV-R-PDSO-G6
- U$5: value SN74LVC2T45 -> SN74LVC1T45; device MyLibrary:DCT-R-PDSO-G8 -> MyLibrary:DBV-R-PDSO-G6
- U2: value MIC5219 3.3V -> MIC5219
- moved U$2 51.5 mm to (0.76, 1.27), flipped to the top, turned to 0 degrees
- moved U$3 48.7 mm to (35.3, 35.3), turned to 270 degrees
- moved J1 41.9 mm to (13.0, 51.6), turned to 0 degrees
- moved C5 39.4 mm to (51.1, 47.0), turned to 270 degrees
- moved C1 39.3 mm to (57.7, 24.9), turned to 270 degrees
- moved U$4 30.3 mm to (35.6, 44.5), flipped to the top, turned to 270 degrees
- moved C7 29.6 mm to (5.84, 47.2), flipped to the bottom, turned to 180 degrees
- moved C3 27.3 mm to (25.9, 36.3), flipped to the top, turned to 180 degrees
- moved R4 26.6 mm to (15.5, 42.2), turned to 90 degrees
- moved C6 22.1 mm to (58.2, 47.0), flipped to the bottom
- moved R3 20.5 mm to (15.7, 35.1), turned to 90 degrees
- moved C2 17.6 mm to (37.1, 48.5), flipped to the top, turned to 0 degrees
- moved XBEE 15.7 mm to (35.6, 24.1), turned to 0 degrees
- moved R1 14.7 mm to (48.5, 24.9), turned to 270 degrees
- moved R2 14.7 mm to (39.6, 13.2), turned to 0 degrees
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- renumbered U$6 to U5
Connections:
- removed net RADIO_OFF: U$5.P$2, U$7.5
- new net RADIO_ON: U$3.P3, U4.5
- net /XBEE_DEBUG: now also R4.1, U$3.P5, U$4.P5; no longer R5.1, U$5.P$5
- net 3.3V: now also C6.1, C8.1, R5.2, U$3.P6, U$4.P6, U$5.P6, U1.1, U3.1, U4.13; no longer C2.1, C3.1, R4.2, U$2.1, U$4.1, U$5.P$8, U$7.13, U$8.P$8
- net 3.3V_ENABLE: now also R1.1, U4.6; no longer R2.1, U$7.6
- net 5V: now also C2.1, C3.1, R1.2, R2.P$2, U$3.P1, U$4.P1, U$5.P1, U4.1; no longer C1.1, C8.1, R1.P$2, R2.2, U$5.P$1, U$7.1, U$8.P$1
- net APDS_9008: now also R6.2, U1.6, U4.10; no longer U$2.6, U$7.11
- net AUX_ANALOG: now also U4.12; no longer U$7.12
- net GND: now also R6.1, U$3.P2, U$4.P2, U$5.P2, U$5.P5, U1.4, U3.3, U3.8, U4.14; no longer U$2.4, U$4.3, U$4.8, U$5.P$4, U$7.14, U$8.P$4, U$8.P$5
- net MISO: now also U4.8; no longer U$7.8
- net MOSI: now also U4.7; no longer U$7.7
- net N$3: now also C1.1; no longer C6.1
- net OPT_101: now also U3.4, U3.5, U4.11; no longer U$4.4, U$4.5, U$7.10
- net RST: now also R4.2, U4.4; no longer R5.2, U$7.4
- net SCK: now also U4.9; no longer U$7.9
- net TINY_RX: now also U$5.P3, U4.2; no longer U$7.2, U$8.P$2
- net TINY_TX: now also U$4.P3, U4.3; no longer U$5.P$3, U$7.3
- net VCC: now also R2.P$1; no longer R1.P$1
- net XBEE_DTR: now also R5.1, U$3.P4; no longer R4.1, U$5.P$7
- net XBEE_RX: now also U$4.P4; no longer U$5.P$6
- net XBEE_TX: now also U$5.P4; no longer U$8.P$7
Routing:
- net 5V: track 110.1 -> 217.6 mm, vias 0 -> 1
- net GND: track 50.0 -> 154.8 mm
- net 3.3V: track 108.1 -> 187.6 mm
- net /XBEE_DEBUG: track 0.00 -> 50.7 mm
- net XBEE_TX: track 0.00 -> 43.8 mm, vias 0 -> 2
- net TINY_RX: track 0.00 -> 40.9 mm, vias 0 -> 2
- net XBEE_RX: track 0.00 -> 34.5 mm, vias 0 -> 2
- net TINY_TX: track 0.00 -> 33.2 mm, vias 0 -> 2
- net 3.3V_ENABLE: track 7.04 -> 40.0 mm, vias 0 -> 2
- net OPT_101: track 0.00 -> 29.5 mm
- net RST: track 0.00 -> 25.3 mm
- net APDS_9008: track 0.00 -> 22.0 mm, vias 0 -> 1
- net MOSI: track 0.00 -> 16.5 mm
- net RADIO_ON: track 0.00 -> 13.8 mm, vias 0 -> 2
- net MISO: track 0.00 -> 13.2 mm
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Other:
- board text added: "ATTINY84"
- board text added: "MM - 02282015 - B"
- board text added: "SOLAR"
- board text removed: "3.3V REGULATOR"
- board text removed: "ATTINY85"
- board text removed: "LEVEL SHIFTER"
- board text removed: "MM - 12192014 - A"
- board text removed: "SOLAR POWER"

Commit message: Grounded USB shield
Parts:
- FRAME1: device SparkFun-Aesthetics:CREATIVE_COMMONS -> MyLibrary:CREATIVE_COMMONS
- moved JP3 0.25 mm to (37.3, 6.10)
Connections:
- net GND: now also JP3.MTN1, JP3.MTN2, JP3.MTN3, JP3.MTN4
Routing:
- net GND: track 154.8 -> 161.4 mm, vias 2 -> 6
Changed lines of the file:
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@@
 <setting verticaltext="up"/>
 </settings>
-<grid distance="0.01" unitdist="inch" unit="inch" style="lines" multiple="1" display="no" altdistance="0.01" altunitdist="inch" altunit="inch"/>
+<grid distance="0.01" unitdist="inch" unit="inch" style="lines" multiple="1" display="no" altdistance="0.005" altunitdist="inch" altunit="inch"/>
 <layers>
-<layer number="1" name="Top" color="4" fill="1" visible="no" active="yes"/>
+<layer number="1" name="Top" color="4" fill="1" visible="yes" active="yes"/>
 <layer number="2" name="Route2" color="1" fill="3" visible="no" active="no"/>
 <layer number="3" name="Route3" color="4" fill="3" visible="no" active="no"/>
@@
 <layer number="19" name="Unrouted" color="6" fill="1" visible="yes" active="yes"/>
 <layer number="20" name="Dimension" color="15" fill="1" visible="yes" active="yes"/>
-<layer number="21" name="tPlace" color="7" fill="1" visible="no" active="yes"/>
-<layer number="22" name="bPlace" color="7" fill="1" visible="no" active="yes"/>
-<layer number="23" name="tOrigins" color="15" fill="1" visible="no" active="yes"/>
+<layer number="21" name="tPlace" color="7" fill="1" visible="yes" active="yes"/>
+<layer number="22" name="bPlace" color="7" fill="1" visible="yes" active="yes"/>
+<layer number="23" name="tOrigins" color="15" fill="1" visible="yes" active="yes"/>
 <layer number="24" name="bOrigins" color="15" fill="1" visible="yes" active="yes"/>
-<layer number="25" name="tNames" color="7" fill="1" visible="no" active="yes"/>
+<layer number="25" name="tNames" color="7" fill="1" visible="yes" active="yes"/>
 <layer number="26" name="bNames" color="7" fill="1" visible="yes" active="yes"/>
 <layer number="27" name="tValues" color="7" fill="1" visible="yes" active="yes"/>
@@
 <text x="7.112" y="30.734" size="1.778" layer="26" rot="MR0">IR</text>
 <text x="68.072" y="7.112" size="1.4224" layer="26" rot="MR0">SUPERCAPACITOR</text>
-<text x="31.496" y="0.508" size="1.016" layer="25" rot="R90">USB POWER</text>
+<text x="45.72" y="0.762" size="1.016" layer="25" rot="R90">USB POWER</text>
 <text x="27.432" y="8.89" size="0.8128" layer="25" rot="R90">DISCHARGE</text>
-<text x="42.926" y="54.356" size="1.27" layer="26" rot="MR0">Autonomous Light Sensor</text>
-<text x="42.926" y="52.578" size="1.27" layer="26" rot="MR0">Cabrillo Robotics Club</text>
-<text x="42.926" y="50.8" size="1.27" layer="26" rot="MR0">MM - 02282015 - B</text>
+<text x="44.704" y="54.356" size="1.27" layer="26" rot="MR0">Autonomous Light Sensor</text>
+<text x="44.704" y="52.578" size="1.27" layer="26" rot="MR0">Cabrillo Robotics Club</text>
+<text x="44.704" y="50.8" size="1.27" layer="26" rot="MR0">MM - 02282015 - B</text>
 <text x="67.31" y="31.75" size="1.778" layer="26" rot="MR0">XBEE</text>
 <text x="67.31" y="31.75" size="1.778" layer="26" rot="MR0">XBEE</text>
@@
 <element name="JP1" library="SparkFun-Connectors" package="1X02_NO_SILK" value="M021X02_NO_SILK" x="65.532" y="26.162" smashed="yes" rot="R270"/>
 <element name="JP2" library="SparkFun-Connectors" package="1X02_NO_SILK" value="M021X02_NO_SILK" x="68.326" y="26.162" smashed="yes" rot="R270"/>
-<element name="JP3" library="SparkFun-Connectors" package="USB-MINIB" value="USBSMD" x="37.592" y="6.096" smashed="yes" rot="R90">
-<attribute name="PROD_ID" value="CONN-08193" x="37.592" y="6.096" size="1.778" layer="27" rot="R90" display="off"/>
-<attribute name="NAME" x="36.322" y="2.286" size="0.4064" layer="25" rot="R90"/>
-<attribute name="VALUE" x="37.592" y="2.286" size="0.4064" layer="27" rot="R90"/>
-</element>
 <element name="R2" library="SparkFun-Passives" package="AXIAL-0.3" value="10" x="39.624" y="13.208" smashed="yes">
 <attribute name="NAME" x="37.846" y="14.986" size="1.27" layer="25" font="vector"/>
 <attribute name="VALUE" x="37.592" y="12.827" size="1.016" layer="21" font="vector" ratio="15"/>
 </element>
-<element name="FRAME1" library="SparkFun-Aesthetics" package="CREATIVE_COMMONS" value="FRAME-LETTER" x="-20.32" y="-10.16"/>
+<element name="FRAME1" library="MyLibrary" package="CREATIVE_COMMONS" value="FRAME-LETTER" x="-20.32" y="-10.16"/>
 <element name="U$2" library="MyLibrary" package="PROTOAREA-10X10" value="PROTOAREA-10X10" x="0.762" y="1.27"/>
 <element name="JP7" library="SparkFun-Connectors" package="1X04_NO_SILK" value="" x="23.622" y="26.67" smashed="yes" rot="R180">
@@
 <element name="R6" library="rcl" package="R1210" value="1k" x="14.986" y="47.498" smashed="yes" rot="MR0">
 <attribute name="NAME" x="19.812" y="46.863" size="1.27" layer="26" rot="MR0"/>
+</element>
+<element name="JP3" library="SparkFun-Connectors" package="USB-MINIB" value="USBSMD" x="37.338" y="6.096" rot="R90">
+<attribute name="PROD_ID" value="CONN-08193" x="37.338" y="6.096" size="1.778" layer="27" rot="R90" display="off"/>
 </element>
 </elements>
@@
 <contactref element="JP1" pad="2"/>
 <contactref element="JP2" pad="2"/>
-<contactref element="JP3" pad="GND"/>
 <contactref element="JP7" pad="1"/>
 <contactref element="JP7" pad="2"/>
@@
 <wire x1="53.086" y1="22.352" x2="53.34" y2="22.098" width="0.6096" layer="1"/>
 <wire x1="53.34" y1="22.098" x2="55.118" y2="22.098" width="0.6096" layer="1"/>
-<wire x1="39.192" y1="8.596" x2="39.192" y2="11.1" width="0.3048" layer="1"/>
-<wire x1="39.192" y1="11.1" x2="39.37" y2="11.176" width="0.3048" layer="1"/>
-<via x="39.37" y="11.176" extent="1-16" drill="0.6" shape="square"/>
+<wire x1="39.192" y1="11.1" x2="39.116" y2="11.176" width="0.3048" layer="1"/>
+<via x="39.116" y="11.176" extent="1-16" drill="0.6" shape="square"/>
 <polygon width="0.3048" layer="16">
 <vertex x="25.146" y="0"/>
@@
 <wire x1="6.4008" y1="52.5272" x2="6.218" y2="52.458" width="0.1524" layer="16"/>
 <wire x1="41.91" y1="24.13" x2="41.91" y2="18.288" width="0.4064" layer="1"/>
-<wire x1="41.91" y1="18.288" x2="41.91" y2="13.716" width="0.4064" layer="1"/>
-<wire x1="41.91" y1="13.716" x2="39.37" y2="11.176" width="0.4064" layer="1"/>
+<wire x1="41.91" y1="18.288" x2="41.91" y2="14.478" width="0.4064" layer="1"/>
+<wire x1="41.91" y1="14.478" x2="39.116" y2="11.176" width="0.4064" layer="1"/>
 <wire x1="23.622" y1="26.67" x2="24.2316" y2="27.2796" width="0.1524" layer="1"/>
 <wire x1="24.2316" y1="36.2712" x2="24.308" y2="36.322" width="0.1524" layer="1"/>
@@
 <wire x1="16.4084" y1="47.498" x2="16.386" y2="47.498" width="0.1524" layer="16"/>
 <wire x1="16.6624" y1="53.4924" x2="16.6116" y2="53.5432" width="0.1524" layer="16"/>
+<contactref element="JP3" pad="MTN2"/>
+<contactref element="JP3" pad="MTN3"/>
+<contactref element="JP3" pad="GND"/>
+<contactref element="JP3" pad="MTN1"/>
+<contactref element="JP3" pad="MTN4"/>
+<via x="31.242" y="8.636" extent="1-16" drill="0.5"/>
+<via x="31.242" y="3.048" extent="1-16" drill="0.5"/>
+<via x="43.434" y="8.636" extent="1-16" drill="0.5"/>
+<via x="43.434" y="3.048" extent="1-16" drill="0.5"/>
+<wire x1="38.938" y1="8.596" x2="39.116" y2="8.85" width="0.4064" layer="1"/>
+<wire x1="39.116" y1="8.85" x2="39.116" y2="11.176" width="0.4064" layer="1"/>
+<wire x1="31.242" y1="8.636" x2="32.838" y2="8.636" width="0.6096" layer="1"/>
+<wire x1="32.838" y1="8.636" x2="32.838" y2="8.596" width="0.6096" layer="1"/>
+<wire x1="31.242" y1="3.048" x2="32.838" y2="3.048" width="0.6096" layer="1"/>
+<wire x1="32.838" y1="3.048" x2="32.838" y2="3.096" width="0.6096" layer="1"/>
+<wire x1="43.434" y1="8.636" x2="41.838" y2="8.636" width="0.6096" layer="1"/>
+<wire x1="41.838" y1="8.636" x2="41.838" y2="8.596" width="0.6096" layer="1"/>
+<wire x1="43.434" y1="3.048" x2="41.838" y2="3.048" width="0.6096" layer="1"/>
+<wire x1="41.838" y1="3.048" x2="41.838" y2="3.096" width="0.6096" layer="1"/>
 </signal>
 <signal name="XBEE_TX">
@@
 <signal name="VCC">
 <contactref element="R2" pad="P$1"/>
-<contactref element="JP3" pad="VBUS"/>
 <contactref element="JP4" pad="1"/>
 <contactref element="TINY" pad="P$4"/>
-<wire x1="35.992" y1="8.596" x2="35.992" y2="13.03" width="0.4064" layer="1"/>
 <wire x1="35.992" y1="13.03" x2="35.814" y2="13.208" width="0.4064" layer="1"/>
 <wire x1="28.702" y1="13.208" x2="35.814" y2="13.208" width="0.4064" layer="1"/>
@@
 <contactref element="XBEE" pad="P$4"/>
 <wire x1="36.83" y1="18.288" x2="36.83" y2="24.13" width="0.4064" layer="1"/>
+<contactref element="JP3" pad="VBUS"/>
+<wire x1="35.992" y1="13.03" x2="35.738" y2="13.03" width="0.4064" layer="1"/>
+<wire x1="35.738" y1="13.03" x2="35.738" y2="8.596" width="0.4064" layer="1"/>
 </signal>
 <signal name="AUX_ANALOG" class="1">

Commit message: Changed pullups to 100K to save power
Parts:
- R1, R5: value 1k -> 100k
Changed lines of the file:
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@@
 <layer number="24" name="bOrigins" color="15" fill="1" visible="yes" active="yes"/>
 <layer number="25" name="tNames" color="7" fill="1" visible="yes" active="yes"/>
-<layer number="26" name="bNames" color="7" fill="1" visible="yes" active="yes"/>
+<layer number="26" name="bNames" color="7" fill="1" visible="no" active="yes"/>
 <layer number="27" name="tValues" color="7" fill="1" visible="yes" active="yes"/>
-<layer number="28" name="bValues" color="7" fill="1" visible="yes" active="yes"/>
+<layer number="28" name="bValues" color="7" fill="1" visible="no" active="yes"/>
 <layer number="29" name="tStop" color="7" fill="3" visible="no" active="yes"/>
 <layer number="30" name="bStop" color="7" fill="6" visible="no" active="yes"/>
@@
 <attribute name="NAME" x="13.843" y="32.512" size="1.27" layer="25" rot="R90"/>
 </element>
-<element name="R5" library="rcl" package="R1210" value="1k" x="42.672" y="31.242" smashed="yes" rot="R270">
+<element name="R5" library="rcl" package="R1210" value="100k" x="42.672" y="31.242" smashed="yes" rot="R270">
 <attribute name="NAME" x="44.577" y="32.512" size="1.27" layer="25" rot="R270"/>
 </element>
@@
 <attribute name="NAME" x="13.589" y="39.624" size="1.27" layer="25" rot="R90"/>
 </element>
-<element name="R1" library="rcl" package="R1210" value="1k" x="48.514" y="24.892" smashed="yes" rot="R270">
+<element name="R1" library="rcl" package="R1210" value="100k" x="48.514" y="24.892" smashed="yes" rot="R270">
 <attribute name="NAME" x="47.498" y="27.559" size="1.27" layer="25"/>
 </element>
